File: disc_finder/disc_finder.kicad_pcb (KiCad board)
At the start: 2 copper layers, 26.5 x 21.1 mm, 22 parts, among them J1 Battery, Q1 DMN6140L-7, Q2 DMN6140L-7, Q3 DMN6140L-7, U1 ICM7555xB, U2 ICM7555xB

Commit message: Limit length of commit hash in rev for dev branch
Other:
- board text added: "-${rev}"
- board text removed: "Rev: ${rev}"
Changed lines of the file:
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@@
 		)
 	)
-	(gr_text "Rev: ${rev}"
-		(at 145.325 109.575 0)
+	(gr_text "-${rev}"
+		(at 139.6 109.65 0)
 		(layer "F.SilkS")
 		(effects
